File: PCB/SAO-display/SAO-display.kicad_pcb (KiCad board)
At the start: 2 copper layers, 69.3 x 80 mm, 49 parts, among them CON1 SAO v1.69bis badge, J1 pogo pins, J2 pads, J3 pogo pins, J4 pads, J5 pogo pins, J6 pads

Commit message: remove some unnecessary vias
Routing:
- net Vin: vias 8 -> 0
Changed lines of the file:
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@@
 			(thermal_bridge_angle 45)
 		)
-		(pad "en" thru_hole roundrect
-			(at 5 -12 270)
-			(size 3 2.2)
-			(drill 0.3
-				(offset -0.5 0)
-			)
-			(layers "*.Cu" "*.Mask")
-			(remove_unused_layers no)
+		(pad "en" smd roundrect
+			(at 5 -12 90)
+			(size 4 2.2)
+			(layers "B.Cu" "B.Mask" "B.Paste")
 			(roundrect_rratio 0.15)
 			(net 4 "enable")
@@
 		(net 1)
 	)
-	(via
-		(at 93.392 118.302)
-		(size 0.6)
-		(drill 0.3)
-		(layers "F.Cu" "B.Cu")
-		(net 2)
-	)
-	(via
-		(at 94.392 118.302)
-		(size 0.6)
-		(drill 0.3)
-		(layers "F.Cu" "B.Cu")
-		(net 2)
-	)
-	(via
-		(at 94.392 116.902)
-		(size 0.6)
-		(drill 0.3)
-		(layers "F.Cu" "B.Cu")
-		(net 2)
-	)
-	(via
-		(at 91.392 116.902)
-		(size 0.6)
-		(drill 0.3)
-		(layers "F.Cu" "B.Cu")
-		(net 2)
-	)
-	(via
-		(at 92.392 118.302)
-		(size 0.6)
-		(drill 0.3)
-		(layers "F.Cu" "B.Cu")
-		(net 2)
-	)
-	(via
-		(at 92.392 116.902)
-		(size 0.6)
-		(drill 0.3)
-		(layers "F.Cu" "B.Cu")
-		(net 2)
-	)
-	(via
-		(at 91.392 118.302)
-		(size 0.6)
-		(drill 0.3)
-		(layers "F.Cu" "B.Cu")
-		(net 2)
-	)
-	(via
-		(at 93.392 116.902)
-		(size 0.6)
-		(drill 0.3)
-		(layers "F.Cu" "B.Cu")
-		(net 2)
-	)
 	(segment
