File: PCB/SAO-display/SAO-display.kicad_pcb (KiCad board)
At the start: 2 copper layers, 69.3 x 80 mm, 49 parts, among them CON1 SAO v1.69bis badge, J1 pogo pins, J2 pads, J3 pogo pins, J4 pads, J5 pogo pins, J6 pads

Commit message: add new front art
Parts:
- added pin: TestPoint_THTPad_D4.0mm_Drill2.0mm, TestPoint:TestPoint_THTPad_D4.0mm_Drill2.0mm, B.Cu at (100.0, 65.0)

Commit message: generated production files
Other:
- board text added: "import SVG scale 0.33"
